Commit message: time experiments added plus an install and run bash

File: data/TROmodels/nao_inertial_python.urdf (robot description, URDF)
Before this commit: robot nao_inertial_python, 25 links, 24 joints
Joints:
- joint Joint1: limit lower=-0.769001 upper=0.397880 effort=0.0 velocity=1.0 -> lower=-0.397880 upper=0.769001 effort=0.0 velocity=1.0
- joint Joint10: limit lower=-1.5446 upper=-0.0349 effort=0.0 velocity=1.0 -> lower=-1.5621 upper=-0.0087 effort=0.0 velocity=1.0
- joint Joint15: limit lower=-1.3265 upper=0.3142 effort=0.0 velocity=1.0 -> lower=-1.6494 upper=-0.0087 effort=0.0 velocity=1.0
- joint Joint17: limit lower=0.0349 upper=1.5446 effort=0.0 velocity=1.0 -> lower=0.0087 upper=1.5621 effort=0.0 velocity=1.0
- joint Joint2: limit lower=-0.922747 upper=1.189516 effort=0.0 velocity=1.0 -> lower=-1.189516 upper=0.922747 effort=0.0 velocity=1.0
- joint Joint3: limit lower=-2.112528 upper=0.092346 effort=0.0 velocity=1.0 -> lower=-0.092346 upper=2.112528 effort=0.0 velocity=1.0
- joint Joint4: limit lower=-0.484090 upper=1.535889 effort=0.0 velocity=1.0 -> lower=-1.535889 upper=0.484090 effort=0.0 velocity=1.0
- joint Joint5: limit lower=-0.790477 upper=0.379472 effort=0.0 velocity=1.0 -> lower=-0.379472 upper=0.790477 effort=0.0 velocity=1.0
- joint Joint8: limit lower=-0.3142 upper=1.3265 effort=0.0 velocity=1.0 -> lower=0.0087 upper=1.6494 effort=0.0 velocity=1.0
- joint joint6: limit lower=-0.740810 upper=1.145303 effort=0.0 velocity=1.0 -> lower=-1.145303 upper=0.740810 effort=0.0 velocity=1.0
